Commit message: chore: misc cleanup (this-session working tree residue)

File: assets/urdf/00-arm-rs_asm-v3/urdf/00-arm-rs_asm-v3.urdf (robot description, URDF)
Before this commit: robot 00-arm-rs_asm-v3, 10 links, 9 joints
Links:
- link base_link: geometry collision mesh filename=meshes/base_link.STL; visual mesh filename=meshes/base_link.STL
- link gripper_end: geometry collision mesh filename=meshes/gripper_end.STL; visual mesh filename=meshes/cnc7.STL
- link gripper_left: geometry collision mesh filename=meshes/gripper_left.STL; visual mesh filename=meshes/cnc_left.STL
- link gripper_right: geometry collision mesh filename=meshes/gripper_right.STL; visual mesh filename=meshes/cnc_right.STL
- link link1: geometry collision mesh filename=meshes/link1.STL; visual mesh filename=meshes/link1.STL
- link link2: mass 1.552 -> 1.972; geometry collision mesh filename=meshes/link2.STL; visual mesh filename=meshes/cnc2.STL
- link link3: mass 1.252 -> 1.062; geometry collision mesh filename=meshes/link3.STL; visual mesh filename=meshes/cnc3.STL
- link link4: mass 0.46 -> 0.66; geometry collision mesh filename=meshes/link4.STL; visual mesh filename=meshes/cnc4.STL
- link link5: mass 0.20120457182895 -> 0.150120457182895; geometry collision mesh filename=meshes/link5.STL; visual mesh filename=meshes/cnc5.STL
- link link6: mass 0.1 -> 0.03; geometry collision mesh filename=meshes/link6.STL; visual mesh filename=meshes/link6.STL
Joints:
- joint joint1: axis 0 0 1 -> 0 0 -1
- joint joint2: axis 0 0 -1 -> 0 0 1; limit lower=-3.14 upper=0 effort=36 velocity=50 -> lower=0 upper=3.14 effort=36 velocity=50
- joint joint3: axis 0 0 1 -> 0 0 -1; limit lower=-3.14 upper=0 effort=36 velocity=50 -> lower=0 upper=3.14 effort=36 velocity=50
- joint joint4: axis 0 0 1 -> 0 0 -1; limit lower=-1.79 upper=1.69 effort=14 velocity=40 -> lower=-1.57 upper=1.57 effort=14 velocity=40
- joint joint5: axis 0 0 1 -> 0 0 -1
- joint joint6: axis 0 0 1 -> 0 0 -1
